File: busy-box.kicad_sch (KiCad schematic)
At the start: 19 parts, among them SW1 SW_SPST, SW2 SW_SPST, SW3 SW_SPST, U1 STM32G030F6Px, U2 LM1117MP-3.3

Commit message: Added sliders
Parts:
- added VR1, VR2, VR3: Alps-Slide-Potentiometer-60mm-RS6011SP6003, rhinocerose-pots:Alps-Slide-Pot-60mm-RS6011SP6003, symbol rhinocerose-interface:Alps-Slide-Potentiometer-60mm-RS6011SP6003
Connections:
- net +3.3V: now also RV1.1, SW1.2 (B), SW2.2 (B), SW3.2 (B), VR1.3 (CW), VR2.3 (CW), VR3.3 (CW)
- net +VDC: no longer SW1.2 (B), SW2.2 (B), SW3.2 (B)
- net GND: now also D1.1 (K), RV1.3, VR1.1 (CCW), VR1.L1 (LUG_TERMINAL_1), VR1.L2 (LUG_TERMINAL_2), VR1.L3 (LUG_TERMINAL_3), VR1.MH1, VR1.MH2, VR2.1 (CCW), VR2.L1 (LUG_TERMINAL_1), VR2.L2 (LUG_TERMINAL_2), VR2.L3 (LUG_TERMINAL_3), VR2.MH1, VR2.MH2, VR3.1 (CCW), VR3.L1 (LUG_TERMINAL_1), VR3.L2 (LUG_TERMINAL_2), VR3.L3 (LUG_TERMINAL_3), VR3.MH1, VR3.MH2
- net ADC_IN_1: now reaches RV1.2
- net ADC_IN_1: now also U1.7 (PA0), VR1.2 (WIPER)
- net ADC_IN_2: now reaches U1.8 (PA1)
- net ADC_IN_2: now also VR2.2 (WIPER)
- net ADC_IN_3: now reaches U1.9 (PA2)
- net ADC_IN_3: now also VR3.2 (WIPER)
